Commit message: August general updates

File: urdf/linorobot.xacro (robot description, xacro)
@@ -1,5 +1,21 @@
- <?xml version="1.0"?>
-   <robot name="linorobot">
-    <link name="base_link">
+<?xml version="1.0"?>
+<robot name="linorobot" xmlns:xacro="http://www.ros.org/wiki/xacro">
+     <link name="base_footprint">
+      <visual>
+        <geometry>
+          <box size="0.21 0.16 0.01"/>
+        </geometry>
+        <origin rpy="0 0 0" xyz="0.0 0.00 0.065"/>
+        <material name="green">
+          <color rgba="0 .8 0 1"/>
+        </material>
+      </visual>
+    </link>
+    <joint name="base_footprint to base_link" type="fixed">
+      <parent link="base_footprint"/>
+      <child link="base_link"/>
+      <origin xyz="0 0 0.098"/>
+    </joint>
+     <link name="base_link">
       <visual>
         <geometry>
@@ -12,5 +28,15 @@
       </visual>
     </link>
-  <link name="imu"/>
+  <link name="imu">
+   <visual>
+        <geometry>
+          <box size="0.21 0.16 0.01"/>
+        </geometry>
+        <origin rpy="0 0 0" xyz="0.0 0.00 0.065"/>
+        <material name="red">
+          <color rgba=".8 0 0 1 "/>
+        </material>
+      </visual>
+    </link>
   <joint name="imu_joint" type="fixed">
   <parent link="base_link"/>
@@ -29,4 +55,50 @@
       </visual>
     </link>
+  <!-- Camera properties -->
+  <joint name="camera_rgb_joint" type="fixed">
+    <parent link="perception_deck" />
+    <child link="camera_rgb_optical_frame" />
+    <origin xyz="0.0 0.0 0.0" rpy="${pi/2} ${pi} ${pi/2}" />
+  </joint>
+  <link name="camera_rgb_optical_frame">
+        <inertial>
+            <origin xyz="0.0 0.0 0.0" rpy="0.0 0.0 0.0" />
+            <mass value="0.00001"/>
+            <inertia
+                ixx="1.0" ixy="0.0"  ixz="0.0"
+                iyy="1.0" iyz="0.0"
+                izz="1.0" />
+        </inertial>
+    </link>
+  <joint name="camera_depth_joint" type="fixed">
+    <parent link="perception_deck" />
+    <child link="camera_depth_optical_frame" />
+    <origin xyz="0.0 0.0 0.0" rpy="${pi/2} ${pi} ${pi/2}" />
+  </joint>
+  <link name="camera_depth_optical_frame" >
+        <inertial>
+            <origin xyz="0.0 0.0 0.0" rpy="0.0 0.0 0.0" />
+            <mass value="0.00001"/>
+            <inertia
+                ixx="1.0" ixy="0.0"  ixz="0.0"
+                iyy="1.0" iyz="0.0"
+                izz="1.0" />
+        </inertial>
+    </link>
+<joint name="camera_depth_frame" type="fixed">
+  <parent link="perception_deck" />
+  <child link="camera_depth_frame_link" />
+  <origin xyz="0.0 0.0 0.0" />
+</joint>
+<link name="camera_depth_frame_link" >
+        <inertial>
+            <origin xyz="0.0 0.0 0.0" rpy="0.0 0.0 0.0" />
+            <mass value="0.00001"/>
+            <inertia
+                ixx="1.0" ixy="0.0"  ixz="0.0"
+                iyy="1.0" iyz="0.0"
+                izz="1.0" />
+        </inertial>
+    </link>
     <link name="wheel_left">
       <visual>
@@ -173,3 +245,3 @@
       <origin xyz="0 0 0"/>
     </joint>
-  </robot>
+</robot>
